File: encoder.sch (KiCad schematic (older format))
At the start: 0 parts

Commit message: Did power and encoder
Parts:
- added C? (x3): 100nF, symbol C
- added C? (x2): 1nF, symbol C
- added R?: 10, symbol R
- added R?: 50, symbol R
- added U?: MLX90365, symbol MLX90365
Connections:
- new net: C?.1, R?.1, U?.1 (VDD)
- new net: C?.2, R?.1, U?.5 (OUT)
- new net: C?.1, U?.7 (VDIG)
- new net +5V: C?.1, R?.2
- new net ENC_OUT: C?.2, R?.2
- new net GND: C?.1, C?.1, C?.2, C?.2, C?.2, U?.2 (Test_x), U?.3 (Test_x), U?.4 (Test_x), U?.6 (Test_x), U?.8 (VSS)
Changed lines of the file:
@@
 LIBS:contrib
 LIBS:valves
-LIBS:testpart
+LIBS:CustomComponents
 LIBS:roller_blade-cache
 EELAYER 25 0
@@
 Comment4 ""
 $EndDescr
+$Comp
+L MLX90365 U?
+U 1 1 5A9ADA9B
+P 3250 3050
+F 0 "U?" H 3250 3350 60  0000 C CNN
+F 1 "MLX90365" H 3250 3450 60  0000 C CNN
+F 2 "" H 3250 3050 60  0001 C CNN
+F 3 "" H 3250 3050 60  0001 C CNN
+	1    3250 3050
+	1    0    0    -1
+$EndComp
+$Comp
+L R R?
+U 1 1 5A9ADC47
+P 2300 2750
+F 0 "R?" V 2380 2750 50  0000 C CNN
+F 1 "10" V 2300 2750 50  0000 C CNN
+F 2 "" V 2230 2750 50  0001 C CNN
+F 3 "" H 2300 2750 50  0001 C CNN
+	1    2300 2750
+	0    1    1    0
+$EndComp
+$Comp
+L C C?
+U 1 1 5A9ADC70
+P 2600 2900
+F 0 "C?" H 2625 3000 50  0000 L CNN
+F 1 "100nF" H 2625 2800 50  0000 L CNN
+F 2 "" H 2638 2750 50  0001 C CNN
+F 3 "" H 2600 2900 50  0001 C CNN
+	1    2600 2900
+	1    0    0    -1
+$EndComp
+$Comp
+L C C?
+U 1 1 5A9ADC92
+P 2600 3300
+F 0 "C?" H 2625 3400 50  0000 L CNN
+F 1 "100nF" H 2625 3200 50  0000 L CNN
+F 2 "" H 2638 3150 50  0001 C CNN
+F 3 "" H 2600 3300 50  0001 C CNN
+	1    2600 3300
+	1    0    0    -1
+$EndComp
+$Comp
+L R R?
+U 1 1 5A9ADD10
+P 2300 3450
+F 0 "R?" V 2380 3450 50  0000 C CNN
+F 1 "50" V 2300 3450 50  0000 C CNN
+F 2 "" V 2230 3450 50  0001 C CNN
+F 3 "" H 2300 3450 50  0001 C CNN
+	1    2300 3450
+	0    1    1    0
+$EndComp
+$Comp
+L C C?
+U 1 1 5A9ADD4B
+P 2000 3300
+F 0 "C?" H 2025 3400 50  0000 L CNN
+F 1 "1nF" H 2025 3200 50  0000 L CNN
+F 2 "" H 2038 3150 50  0001 C CNN
+F 3 "" H 2000 3300 50  0001 C CNN
+	1    2000 3300
+	1    0    0    -1
+$EndComp
+$Comp
+L C C?
+U 1 1 5A9ADD85
+P 2000 2900
+F 0 "C?" H 2025 3000 50  0000 L CNN
+F 1 "1nF" H 2025 2800 50  0000 L CNN
+F 2 "" H 2038 2750 50  0001 C CNN
+F 3 "" H 2000 2900 50  0001 C CNN
+	1    2000 2900
+	1    0    0    -1
+$EndComp
+$Comp
+L GND #PWR?
+U 1 1 5A9ADF2A
+P 1800 3100
+F 0 "#PWR?" H 1800 2850 50  0001 C CNN
+F 1 "GND" H 1800 2950 50  0000 C CNN
+F 2 "" H 1800 3100 50  0001 C CNN
+F 3 "" H 1800 3100 50  0001 C CNN
+	1    1800 3100
+	1    0    0    -1
+$EndComp
+$Comp
+L +5V #PWR?
+U 1 1 5A9AE4C6
+P 2000 2750
+F 0 "#PWR?" H 2000 2600 50  0001 C CNN
+F 1 "+5V" H 2000 2890 50  0000 C CNN
+F 2 "" H 2000 2750 50  0001 C CNN
+F 3 "" H 2000 2750 50  0001 C CNN
+	1    2000 2750
+	1    0    0    -1
+$EndComp
+Text HLabel 2000 3450 0    60   Input ~ 0
+ENC_OUT
+$Comp
+L GND #PWR?
+U 1 1 5A9AEA7E
+P 4000 3200
+F 0 "#PWR?" H 4000 2950 50  0001 C CNN
+F 1 "GND" H 4000 3050 50  0000 C CNN
+F 2 "" H 4000 3200 50  0001 C CNN
+F 3 "" H 4000 3200 50  0001 C CNN
+	1    4000 3200
+	1    0    0    -1
+$EndComp
+Wire Wire Line
+	1800 3100 2800 3100
+Wire Wire Line
+	2600 3050 2600 3150
+Connection ~ 2600 3100
+Wire Wire Line
+	2800 3450 2800 3300
+Wire Wire Line
+	2450 3450 2800 3450
+Wire Wire Line
+	2800 2750 2800 2900
+Wire Wire Line
+	2450 2750 2800 2750
+Connection ~ 2600 2750
+Connection ~ 2600 3450
+Wire Wire Line
+	2150 3450 2000 3450
+Wire Wire Line
+	2150 2750 2000 2750
+Wire Wire Line
+	2000 3050 2000 3150
+Connection ~ 2000 3100
+Wire Wire Line
+	3750 2900 3750 3200
+Connection ~ 3750 3000
+Connection ~ 3750 3100
+Wire Wire Line
+	3750 3200 4000 3200
+$Comp
+L C C?
+U 1 1 5A9AEC0C
+P 3750 3550
+F 0 "C?" H 3775 3650 50  0000 L CNN
+F 1 "100nF" H 3775 3450 50  0000 L CNN
+F 2 "" H 3788 3400 50  0001 C CNN
+F 3 "" H 3750 3550 50  0001 C CNN
+	1    3750 3550
+	1    0    0    -1
+$EndComp
+Wire Wire Line
+	3750 3350 3750 3400
+$Comp
+L GND #PWR?
+U 1 1 5A9AEC74
+P 3750 3700
+F 0 "#PWR?" H 3750 3450 50  0001 C CNN
+F 1 "GND" H 3750 3550 50  0000 C CNN
+F 2 "" H 3750 3700 50  0001 C CNN
+F 3 "" H 3750 3700 50  0001 C CNN
+	1    3750 3700
+	1    0    0    -1
+$EndComp
 $EndSCHEMATC
