File: FS.sch (KiCad schematic (older format))
At the start: 0 parts

Commit message: adding blade connector pcb
Parts:
- added J1: Conn_01x02, symbol Conn_01x02
Connections:
- net labels added: +12V, GND
- wire segments 0 -> 1
Changed lines of the file:
@@
 LIBS:contrib
 LIBS:valves
-LIBS:CustomComponents
-LIBS:roller_blade-cache
 EELAYER 25 0
 EELAYER END
 $Descr A4 11693 8268
 encoding utf-8
-Sheet 1 6
+Sheet 1 1
 Title ""
 Date ""
@@
 Comment4 ""
 $EndDescr
+$Comp
+L Conn_01x02 J1
+U 1 1 5AC9316A
+P 2900 2100
+F 0 "J1" H 2900 2200 50  0000 C CNN
+F 1 "Conn_01x02" H 2900 1900 50  0000 C CNN
+F 2 "" H 2900 2100 50  0001 C CNN
+F 3 "" H 2900 2100 50  0001 C CNN
+	1    2900 2100
+	1    0    0    -1
+$EndComp
+$Comp
+L +12V #PWR?
+U 1 1 5AC93321
+P 2700 2100
+F 0 "#PWR?" H 2700 1950 50  0001 C CNN
+F 1 "+12V" H 2700 2240 50  0000 C CNN
+F 2 "" H 2700 2100 50  0001 C CNN
+F 3 "" H 2700 2100 50  0001 C CNN
+	1    2700 2100
+	1    0    0    -1
+$EndComp
+Wire Wire Line
+	2700 2200 2600 2200
+$Comp
+L GND #PWR?
+U 1 1 5AC93386
+P 2600 2200
+F 0 "#PWR?" H 2600 1950 50  0001 C CNN
+F 1 "GND" H 2600 2050 50  0000 C CNN
+F 2 "" H 2600 2200 50  0001 C CNN
+F 3 "" H 2600 2200 50  0001 C CNN
+	1    2600 2200
+	1    0    0    -1
+$EndComp
 $EndSCHEMATC
