File: RecieverAndController/reciever_mod.sch (KiCad schematic (older format))
At the start: 24 parts

Commit message: Waiting for the merge conflict storm
Parts:
- C1: value 4.7pF -> 2.7pF
- L1: value 100nH -> 47nH
- L2: value 27nH -> 15nH
- Y?: renamed from 9.8375MHz; value Crystal -> 13.56MHz
Changed lines of the file:
@@
 P 5000 3500
 F 0 "U?" H 5000 3500 60  0000 C CNN
-F 1 "MAX7036" H 5000 3500 60  0000 C CNN
+F 1 "MAX7036" H 5000 3600 60  0000 C CNN
 F 2 "" H 5000 3500 60  0001 C CNN
 F 3 "" H 5000 3500 60  0001 C CNN
@@
 P 5550 4900
 F 0 "L1" V 5500 4900 50  0000 C CNN
-F 1 "100nH" V 5625 4900 50  0000 C CNN
+F 1 "47nH" V 5625 4900 50  0000 C CNN
 F 2 "" H 5550 4900 50  0001 C CNN
 F 3 "" H 5550 4900 50  0001 C CNN
@@
 $EndComp
 $Comp
-L Crystal 9.8375MHz
+L Crystal Y?
 U 1 1 5A9AD39F
 P 4900 4850
-F 0 "9.8375MHz" H 4900 5000 50  0000 C CNN
-F 1 "Crystal" H 4900 4700 50  0000 C CNN
+F 0 "Y?" H 4900 5000 50  0000 C CNN
+F 1 "13.56MHz" H 4900 4700 50  0000 C CNN
 F 2 "" H 4900 4850 50  0001 C CNN
 F 3 "" H 4900 4850 50  0001 C CNN
@@
 P 2450 3600
 F 0 "R2" V 2530 3600 50  0000 C CNN
-F 1 "220kOhm" V 2450 3600 50  0000 C CNN
+F 1 "220kOhm" V 2350 3600 50  0000 C CNN
 F 2 "" V 2380 3600 50  0001 C CNN
 F 3 "" H 2450 3600 50  0001 C CNN
@@
 P 6000 4050
 F 0 "C1" H 6025 4150 50  0000 L CNN
-F 1 "4.7pF" H 6025 3950 50  0000 L CNN
+F 1 "2.7pF" H 6025 3950 50  0000 L CNN
 F 2 "" H 6038 3900 50  0001 C CNN
 F 3 "" H 6000 4050 50  0001 C CNN
@@
 P 7000 3900
 F 0 "L2" V 6950 3900 50  0000 C CNN
-F 1 "27nH" V 7075 3900 50  0000 C CNN
+F 1 "15nH" V 7075 3900 50  0000 C CNN
 F 2 "" H 7000 3900 50  0001 C CNN
 F 3 "" H 7000 3900 50  0001 C CNN
