File: RecieverAndController/reciever_mod.sch (KiCad schematic (older format))
At the start: 24 parts, among them U2 MAX7036, Y2 13.56MHz

Commit message: Finished transmitter
Parts:
- C1: footprint (none) -> Capacitors_SMD:C_0603
- L1, L2: footprint (none) -> Inductors_SMD:L_0603
Changed lines of the file:
@@
 F 0 "L1" V 5500 4900 50  0000 C CNN
 F 1 "47nH" V 5625 4900 50  0000 C CNN
-F 2 "" H 5550 4900 50  0001 C CNN
+F 2 "Inductors_SMD:L_0603" H 5550 4900 50  0001 C CNN
 F 3 "" H 5550 4900 50  0001 C CNN
 	1    5550 4900
@@
 F 0 "C1" H 6025 4150 50  0000 L CNN
 F 1 "2.7pF" H 6025 3950 50  0000 L CNN
-F 2 "" H 6038 3900 50  0001 C CNN
+F 2 "Capacitors_SMD:C_0603" H 6038 3900 50  0001 C CNN
 F 3 "" H 6000 4050 50  0001 C CNN
 	1    6000 4050
@@
 F 0 "L2" V 6950 3900 50  0000 C CNN
 F 1 "15nH" V 7075 3900 50  0000 C CNN
-F 2 "" H 7000 3900 50  0001 C CNN
+F 2 "Inductors_SMD:L_0603" H 7000 3900 50  0001 C CNN
 F 3 "" H 7000 3900 50  0001 C CNN
 	1    7000 3900
