File: RecieverAndController/_saved_encoder.sch (KiCad schematic (older format))
At the start: 8 parts, among them U3 MLX90365

Commit message: adding start of pcb
Parts:
- added J3, J4: Conn_01x03, Pin_Headers:Pin_Header_Angled_1x03_Pitch2.54mm, symbol Conn_01x03
Connections:
- net +5V: now also J4.1 (Pin_1); no longer C24.1, R4.2
- net ENC_OUT: now also J4.2 (Pin_2); no longer C25.2, R5.2
- net GND: now also J4.3 (Pin_3); no longer C24.2, C25.1, C26.2, C27.1, C28.2, U3.2 (Test_x), U3.3 (Test_x), U3.4 (Test_x), U3.6 (Test_x), U3.8 (VSS)
- new net 5V_L: C24.1, J3.1 (Pin_1), R4.2
- new net ENC_OUT_L: C25.2, J3.2 (Pin_2), R5.2
- new net GND_L: C24.2, C25.1, C26.2, C27.1, C28.2, J3.3 (Pin_3), U3.2 (Test_x), U3.3 (Test_x), U3.4 (Test_x), U3.6 (Test_x), U3.8 (VSS)
Changed lines of the file:
@@
-$EndComp
-$Comp
-L C C25
-U 1 1 5A9ADD4B
-P 2000 3300
-F 0 "C25" H 2025 3400 50  0000 L CNN
-F 1 "1nF" H 2025 3200 50  0000 L CNN
-F 2 "Capacitors_SMD:C_0603" H 2038 3150 50  0001 C CNN
-F 3 "" H 2000 3300 50  0001 C CNN
-	1    2000 3300
-	1    0    0    -1
 $EndComp
 $Comp
@@
 F 3 "" H 2000 2900 50  0001 C CNN
 	1    2000 2900
-	1    0    0    -1
-$EndComp
-$Comp
-L GND #PWR031
-U 1 1 5A9ADF2A
-P 1800 3100
-F 0 "#PWR031" H 1800 2850 50  0001 C CNN
-F 1 "GND" H 1800 2950 50  0000 C CNN
-F 2 "" H 1800 3100 50  0001 C CNN
-F 3 "" H 1800 3100 50  0001 C CNN
-	1    1800 3100
-	1    0    0    -1
-$EndComp
-$Comp
-L +5V #PWR032
-U 1 1 5A9AE4C6
-P 2000 2750
-F 0 "#PWR032" H 2000 2600 50  0001 C CNN
-F 1 "+5V" H 2000 2890 50  0000 C CNN
-F 2 "" H 2000 2750 50  0001 C CNN
-F 3 "" H 2000 2750 50  0001 C CNN
-	1    2000 2750
-	1    0    0    -1
-$EndComp
-Text HLabel 2000 3450 0    60   Input ~ 0
-ENC_OUT
-$Comp
-L GND #PWR033
-U 1 1 5A9AEA7E
-P 4000 3200
-F 0 "#PWR033" H 4000 2950 50  0001 C CNN
-F 1 "GND" H 4000 3050 50  0000 C CNN
-F 2 "" H 4000 3200 50  0001 C CNN
-F 3 "" H 4000 3200 50  0001 C CNN
-	1    4000 3200
 	1    0    0    -1
 $EndComp
@@
 	3750 3350 3750 3400
 $Comp
-L GND #PWR034
-U 1 1 5A9AEC74
-P 3750 3700
-F 0 "#PWR034" H 3750 3450 50  0001 C CNN
-F 1 "GND" H 3750 3550 50  0000 C CNN
-F 2 "" H 3750 3700 50  0001 C CNN
-F 3 "" H 3750 3700 50  0001 C CNN
-	1    3750 3700
+L Conn_01x03 J3
+U 1 1 5ACAF373
+P 4650 2800
+F 0 "J3" H 4650 3000 50  0000 C CNN
+F 1 "Conn_01x03" H 4650 2600 50  0000 C CNN
+F 2 "Pin_Headers:Pin_Header_Angled_1x03_Pitch2.54mm" H 4650 2800 50  0001 C CNN
+F 3 "" H 4650 2800 50  0001 C CNN
+	1    4650 2800
 	1    0    0    -1
 $EndComp
+Text Label 4450 2900 2    60   ~ 0
+GND_L
+Text Label 4450 2800 2    60   ~ 0
+ENC_OUT_L
+Text Label 4450 2700 2    60   ~ 0
+5V_L
+Text Label 2000 2750 2    60   ~ 0
+5V_L
+$Comp
+L C C25
+U 1 1 5A9ADD4B
+P 2000 3300
+F 0 "C25" H 2025 3400 50  0000 L CNN
+F 1 "1nF" H 2025 3200 50  0000 L CNN
+F 2 "Capacitors_SMD:C_0603" H 2038 3150 50  0001 C CNN
+F 3 "" H 2000 3300 50  0001 C CNN
+	1    2000 3300
+	1    0    0    -1
+$EndComp
+Text Label 1800 3100 2    60   ~ 0
+GND_L
+Text Label 4000 3200 3    60   ~ 0
+GND_L
+Text Label 3750 3700 2    60   ~ 0
+GND_L
+Text Label 2000 3450 2    60   ~ 0
+ENC_OUT_L
+$Comp
+L Conn_01x03 J4
+U 1 1 5ACAF700
+P 5550 2800
+F 0 "J4" H 5550 3000 50  0000 C CNN
+F 1 "Conn_01x03" H 5850 2800 50  0000 C CNN
+F 2 "Pin_Headers:Pin_Header_Angled_1x03_Pitch2.54mm" H 5550 2800 50  0001 C CNN
+F 3 "" H 5550 2800 50  0001 C CNN
+	1    5550 2800
+	1    0    0    -1
+$EndComp
+Text HLabel 5350 2800 0    60   Input ~ 0
+ENC_OUT
+$Comp
+L GND #PWR031
+U 1 1 5ACAF7BE
+P 5350 2900
+F 0 "#PWR031" H 5350 2650 50  0001 C CNN
+F 1 "GND" H 5350 2750 50  0000 C CNN
+F 2 "" H 5350 2900 50  0001 C CNN
+F 3 "" H 5350 2900 50  0001 C CNN
+	1    5350 2900
+	1    0    0    -1
+$EndComp
+$Comp
+L +5V #PWR032
+U 1 1 5ACAF7E6
+P 5350 2700
+F 0 "#PWR032" H 5350 2550 50  0001 C CNN
+F 1 "+5V" H 5350 2840 50  0000 C CNN
+F 2 "" H 5350 2700 50  0001 C CNN
+F 3 "" H 5350 2700 50  0001 C CNN
+	1    5350 2700
+	1    0    0    -1
+$EndComp
