File: Transmitter/Transmitter.sch (KiCad schematic (older format))
At the start: 25 parts, among them U1 MAX7044, Y1 13.56MHz

Commit message: Finished transmitter
Parts:
- removed Y1: 13.56MHz, symbol Crystal
- added D1: LED, LEDs:LED_0805, symbol LED
- added R2: 100, Resistors_SMD:R_0603, symbol R
- added Y1: 13.56MHz, Custom:1253-1737-1-ND, symbol Crystal_GND24
- AE1: footprint (none) -> Custom:311-1570-1-ND
- BT1: renamed from BT?; footprint (none) -> Battery_Holders:Keystone_3034_1x20mm-CoinCell
- C1, C10, C11, C12, C13, C5, C8, C9: renamed from C?; footprint (none) -> Capacitors_SMD:C_0603
- C2, C3, C4, C6, C7: footprint (none) -> Capacitors_SMD:C_0603
- L1, L2: footprint (none) -> Inductors_SMD:L_0603
- L3: renamed from L?; footprint (none) -> Inductors_SMD:L_0603
- R1: renamed from R?; footprint (none) -> Resistors_SMD:R_0603
- RV1: renamed from RV?; footprint (none) -> Custom:254TA103B50A
- U1: footprint (none) -> TO_SOT_Packages_SMD:SOT-23-8
- U2: renamed from U?; footprint (none) -> TO_SOT_Packages_SMD:TSOT-23-6
- U3: renamed from U?; footprint (none) -> Housings_SSOP:VSSOP-8_3.0x3.0mm_Pitch0.65mm
- Y2: renamed from Y?; value 1MHz -> 3MHz; footprint (none) -> Custom:ABLS-LR-3.000MHZ-T
Connections:
- net +3V3: now also D1.2 (A)
- net GND: now also R2.2, Y1.2, Y1.4
- net at C5.2, U1.1 (XTAL1): now also Y1.1
- net at C9.2, U1.8 (XTAL2): now also Y1.3
- new net: D1.1 (K), R2.1
